File: BLV_PCB.kicad_pcb (KiCad board)
At the start: 4 copper layers, 90 x 90 mm, 96 parts, among them J1 JST-PH, J10 USB_C_USB2.0_16P, J11 Micro_SD_Card, J12 duPont, J2 JST-PH, J3 JST-PH, J4 duPont, J5 duPont, J6 duPont, J8 USB_C_USB2.0_16P, Q1 Si2301CDS, Q2 Si2301CDS, SW11 SW_QSPI, SW12 SW_RUN, SW3 SW_GNSS, U11 W25Q128JVS, U12 RP2350_60QFN, U3 TPS63001DRCR, U4 BH-18650-A6AJ012, U5 E32-400M30S, U6 NEO-M9N, Y11 ABM8_262_T3

Commit message: BLV PCB v0.2
Parts:
- removed TP2: +3V3, TestPoint:TestPoint_Pad_D1.0mm
- TP4: moved to F.Cu
- moved TP4 91.1 mm to (192.1, 43.7)
- moved TP3 9.58 mm to (187.2, 61.8)
Routing:
- net +3V3: track 62.1 -> 59.7 mm, vias 44 -> 42
- net /GNSS & MicroSD/SPI_CS1: track 38.2 -> 37.5 mm
- net GND: vias 334 -> 333
