File: MCU.kicad_sch (KiCad schematic)
At the start: 44 parts, among them J7 duPont, SW1 SW_QSPI, SW2 SW_RUN, U1 W25Q128JVS, U2 RP2350_60QFN, Y1 ABM8_262_T3

Commit message: BLV PCB v0.2
Parts:
- renumbered C1 to C11, C2 to C12, C3 to C13, C4 to C14, C5 to C15, C6 to C16, C7 to C17, C8 to C18, C9 to C19, C10 to C20, C11 to C21, C12 to C22, C13 to C23, C14 to C24, C15 to C25, C16 to C26, D1 to D11, D2 to D12, D3 to D13, J7 to J12, L1 to L11, R1 to R11, R2 to R12, R3 to R13, R4 to R14, R5 to R15, R6 to R16, R7 to R17, R19 to R18, R20 to R19, R21 to R20, R8 to R21, R28 to R23, R29 to R24, R9 to R25, R12 to R26, R13 to R27, R14 to R28, SW1 to SW11, SW2 to SW12, U1 to U11, U2 to U12, Y1 to Y11
Other:
- moved on the sheet: D11, D12, D13, R26, R27, R28
